File: soc_core_power.kicad_sch (KiCad schematic)
At the start: 2 parts

Commit message: write some things down
Parts:
- U1: renamed from U?; value MCIMX6YxxVMxxxx -> MCIMX6Y2DVM09AB; Manufacturer (none) -> NXP; MfgPartNo (none) -> MCIMX6Y2DVM09AB; Vendor (none) -> Digi-Key; VendorPartNo (none) -> 568-14995-ND
Other:
- note added: "onoff/PoR test points bootmode test points"
- note removed: "TODO: UART header"
Changed lines of the file:
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@@
     (company "Ian Kilgore")
   )
-  (text "TODO: UART header" (at 43.18 46.99 0)
+  (text "onoff/PoR test points\nbootmode test points" (at 43.18 46.99 0)
     (effects (font (size 1.27 1.27)) (justify left bottom))
   )
   (symbol (lib_id "catfood:MCIMX6YxxVMxxxx") (at 99.06 62.23 0) (unit 1)
     (in_bom yes) (on_board yes) (fields_autoplaced)
-    (property "Reference" "U?" (id 0) (at 99.06 31.75 0))
-    (property "Value" "MCIMX6YxxVMxxxx" (id 1) (at 99.06 34.29 0))
+    (property "Reference" "U1" (id 0) (at 99.06 30.48 0))
+    (property "Value" "MCIMX6Y2DVM09AB" (id 1) (at 99.06 33.02 0))
     (property "Footprint" "" (id 2) (at 88.9 43.18 0)
       (effects (font (size 1.27 1.27)) hide)
     )
     (property "Datasheet" "" (id 3) (at 88.9 43.18 0)
+      (effects (font (size 1.27 1.27)) hide)
+    )
+    (property "Manufacturer" "NXP" (id 4) (at 99.06 41.91 0)
+      (effects (font (size 1.27 1.27)) hide)
+    )
+    (property "MfgPartNo" "MCIMX6Y2DVM09AB" (id 5) (at 99.06 44.45 0)
+      (effects (font (size 1.27 1.27)) hide)
+    )
+    (property "Vendor" "Digi-Key" (id 6) (at 99.06 46.99 0)
+      (effects (font (size 1.27 1.27)) hide)
+    )
+    (property "VendorPartNo" "568-14995-ND" (id 7) (at 99.06 49.53 0)
       (effects (font (size 1.27 1.27)) hide)
     )
@@
   (symbol (lib_id "catfood:MCIMX6YxxVMxxxx") (at 153.67 57.15 0) (unit 2)
     (in_bom yes) (on_board yes) (fields_autoplaced)
-    (property "Reference" "U?" (id 0) (at 151.13 27.94 0))
-    (property "Value" "MCIMX6YxxVMxxxx" (id 1) (at 151.13 30.48 0))
+    (property "Reference" "U1" (id 0) (at 151.13 27.94 0))
+    (property "Value" "MCIMX6Y2DVM09AB" (id 1) (at 151.13 30.48 0))
     (property "Footprint" "" (id 2) (at 143.51 38.1 0)
       (effects (font (size 1.27 1.27)) hide)
@@
       (effects (font (size 1.27 1.27)) hide)
     )
+    (property "Manufacturer" "NXP" (id 4) (at 151.13 38.1 0)
+      (effects (font (size 1.27 1.27)) hide)
+    )
+    (property "MfgPartNo" "MCIMX6Y2DVM09AB" (id 5) (at 151.13 40.64 0)
+      (effects (font (size 1.27 1.27)) hide)
+    )
+    (property "Vendor" "Digi-Key" (id 6) (at 151.13 43.18 0)
+      (effects (font (size 1.27 1.27)) hide)
+    )
+    (property "VendorPartNo" "568-14995-ND" (id 7) (at 151.13 45.72 0)
+      (effects (font (size 1.27 1.27)) hide)
+    )
