File: soc_core_power.kicad_sch (KiCad schematic)
At the start: 19 parts, among them U4 MCIMX6Y2DVM09AB

Commit message: ERC: power flags
Changed lines of the file:
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@@
   (junction (at 163.83 87.63) (diameter 0) (color 0 0 0 0)
   )
+  (junction (at 174.625 102.87) (diameter 0) (color 0 0 0 0)
+  )
   (junction (at 186.69 102.87) (diameter 0) (color 0 0 0 0)
   )
@@
     (stroke (width 0) (type default) (color 0 0 0 0))
   )
-  (wire (pts (xy 168.91 102.87) (xy 186.69 102.87))
+  (wire (pts (xy 168.91 102.87) (xy 174.625 102.87))
     (stroke (width 0) (type default) (color 0 0 0 0))
   )
@@
     (stroke (width 0) (type default) (color 0 0 0 0))
   )
+  (wire (pts (xy 174.625 102.87) (xy 186.69 102.87))
+    (stroke (width 0) (type default) (color 0 0 0 0))
+  )
   (wire (pts (xy 199.39 78.74) (xy 199.39 80.01))
     (stroke (width 0) (type default) (color 0 0 0 0))
@@
   )
   (wire (pts (xy 199.39 87.63) (xy 199.39 90.17))
+    (stroke (width 0) (type default) (color 0 0 0 0))
+  )
+  (wire (pts (xy 174.625 101.6) (xy 174.625 102.87))
     (stroke (width 0) (type default) (color 0 0 0 0))
   )
@@
       (effects (font (size 1.27 1.27)) hide)
     )
+    (pin "1")
+  )
+  (symbol (lib_id "power:PWR_FLAG") (at 174.625 101.6 0) (unit 1)
+    (in_bom yes) (on_board yes)
+    (property "Reference" "#FLG0101" (id 0) (at 174.625 99.695 0)
+      (effects (font (size 1.27 1.27)) hide)
+    )
+    (property "Value" "PWR_FLAG" (id 1) (at 174.625 97.79 0))
+    (property "Footprint" "" (id 2) (at 174.625 101.6 0)
+      (effects (font (size 1.27 1.27)) hide)
+    )
+    (property "Datasheet" "~" (id 3) (at 174.625 101.6 0)
+      (effects (font (size 1.27 1.27)) hide)
+    )

Commit message: Footprint assignments for standard passives
Parts:
- C15, C29, C30, C31, C32: footprint (none) -> Capacitor_SMD:C_0805_2012Metric
- C16, C18: footprint (none) -> Capacitor_SMD:C_0603_1608Metric
- C17, C19, C20, C21, C22, C23, C24, C25, C26, C27, C28: footprint (none) -> Capacitor_SMD:C_0402_1005Metric
Changed lines of the file:
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@@
       (effects (font (size 1.27 1.27)) (justify left))
     )
-    (property "Footprint" "" (id 2) (at 110.49 92.71 0)
+    (property "Footprint" "Capacitor_SMD:C_0402_1005Metric" (id 2) (at 110.49 92.71 0)
       (effects (font (size 1.27 1.27)) hide)
     )
@@
       (effects (font (size 1.27 1.27)) (justify left))
     )
-    (property "Footprint" "" (id 2) (at 186.69 107.95 0)
+    (property "Footprint" "Capacitor_SMD:C_0805_2012Metric" (id 2) (at 186.69 107.95 0)
       (effects (font (size 1.27 1.27)) hide)
     )
@@
       (effects (font (size 1.27 1.27)) (justify left))
     )
-    (property "Footprint" "" (id 2) (at 163.83 74.93 0)
+    (property "Footprint" "Capacitor_SMD:C_0402_1005Metric" (id 2) (at 163.83 74.93 0)
       (effects (font (size 1.27 1.27)) hide)
     )
@@
       (effects (font (size 1.27 1.27)) (justify left))
     )
-    (property "Footprint" "" (id 2) (at 163.83 92.71 0)
+    (property "Footprint" "Capacitor_SMD:C_0402_1005Metric" (id 2) (at 163.83 92.71 0)
       (effects (font (size 1.27 1.27)) hide)
     )
@@
       (effects (font (size 1.27 1.27)) (justify left))
     )
-    (property "Footprint" "" (id 2) (at 184.15 127 0)
+    (property "Footprint" "Capacitor_SMD:C_0805_2012Metric" (id 2) (at 184.15 127 0)
       (effects (font (size 1.27 1.27)) hide)
     )
@@
       (effects (font (size 1.27 1.27)) (justify left))
     )
-    (property "Footprint" "" (id 2) (at 168.91 107.95 0)
+    (property "Footprint" "Capacitor_SMD:C_0402_1005Metric" (id 2) (at 168.91 107.95 0)
       (effects (font (size 1.27 1.27)) hide)
     )
@@
       (effects (font (size 1.27 1.27)) (justify left))
     )
-    (property "Footprint" "" (id 2) (at 76.2 74.93 0)
+    (property "Footprint" "Capacitor_SMD:C_0603_1608Metric" (id 2) (at 76.2 74.93 0)
       (effects (font (size 1.27 1.27)) hide)
     )
@@
       (effects (font (size 1.27 1.27)) (justify left))
     )
-    (property "Footprint" "" (id 2) (at 166.37 127 0)
+    (property "Footprint" "Capacitor_SMD:C_0402_1005Metric" (id 2) (at 166.37 127 0)
       (effects (font (size 1.27 1.27)) hide)
     )
@@
       (effects (font (size 1.27 1.27)) (justify left))
     )
-    (property "Footprint" "" (id 2) (at 110.49 74.93 0)
+    (property "Footprint" "Capacitor_SMD:C_0402_1005Metric" (id 2) (at 110.49 74.93 0)
       (effects (font (size 1.27 1.27)) hide)
     )
@@
       (effects (font (size 1.27 1.27)) (justify left))
     )
-    (property "Footprint" "" (id 2) (at 181.61 74.93 0)
+    (property "Footprint" "Capacitor_SMD:C_0402_1005Metric" (id 2) (at 181.61 74.93 0)
       (effects (font (size 1.27 1.27)) hide)
     )
@@
       (effects (font (size 1.27 1.27)) (justify left))
     )
-    (property "Footprint" "" (id 2) (at 199.39 74.93 0)
+    (property "Footprint" "Capacitor_SMD:C_0805_2012Metric" (id 2) (at 199.39 74.93 0)
       (effects (font (size 1.27 1.27)) hide)
     )
@@
       (effects (font (size 1.27 1.27)) (justify left))
     )
-    (property "Footprint" "" (id 2) (at 162.56 138.43 0)
+    (property "Footprint" "Capacitor_SMD:C_0402_1005Metric" (id 2) (at 162.56 138.43 0)
       (effects (font (size 1.27 1.27)) hide)
     )
@@
       (effects (font (size 1.27 1.27)) (justify left))
     )
-    (property "Footprint" "" (id 2) (at 92.71 74.93 0)
+    (property "Footprint" "Capacitor_SMD:C_0402_1005Metric" (id 2) (at 92.71 74.93 0)
       (effects (font (size 1.27 1.27)) hide)
     )
@@
       (effects (font (size 1.27 1.27)) (justify left))
     )
-    (property "Footprint" "" (id 2) (at 199.39 92.71 0)
+    (property "Footprint" "Capacitor_SMD:C_0805_2012Metric" (id 2) (at 199.39 92.71 0)
       (effects (font (size 1.27 1.27)) hide)
     )
@@
       (effects (font (size 1.27 1.27)) (justify left))
     )
-    (property "Footprint" "" (id 2) (at 181.61 92.71 0)
+    (property "Footprint" "Capacitor_SMD:C_0402_1005Metric" (id 2) (at 181.61 92.71 0)
       (effects (font (size 1.27 1.27)) hide)
     )
@@
       (effects (font (size 1.27 1.27)) (justify left))
     )
-    (property "Footprint" "" (id 2) (at 59.69 74.93 0)
+    (property "Footprint" "Capacitor_SMD:C_0805_2012Metric" (id 2) (at 59.69 74.93 0)
       (effects (font (size 1.27 1.27)) hide)
     )
@@
       (effects (font (size 1.27 1.27)) (justify left))
     )
-    (property "Footprint" "" (id 2) (at 93.98 92.71 0)
+    (property "Footprint" "Capacitor_SMD:C_0603_1608Metric" (id 2) (at 93.98 92.71 0)
       (effects (font (size 1.27 1.27)) hide)
     )
@@
       (effects (font (size 1.27 1.27)) (justify left))
     )
-    (property "Footprint" "" (id 2) (at 93.98 106.68 0)
-      (effects (font (size 1.27 1.27)) hide)
-    )
+    (property "Footprint" "Capacitor_SMD:C_0402_1005Metric" (id 2) (at 93.98 106.68 0)
+      (effects (font (size 1.27 1.27)) hide)
+    )
