File: soc_core_power.kicad_sch (KiCad schematic)
At the start: 19 parts, among them U4 MCIMX6Y2DVM09AB

Commit message: Update fields
Parts:
- C15, C31, C32: Manufacturer (none) -> Murata Electronics; MfgPartNo (none) -> GRM21BR61A226ME51L; Vendor (none) -> Digi-Key; VendorPartNo (none) -> 490-10511-1-ND
- C16, C18: Manufacturer (none) -> Samsung Electro-Mechanics; MfgPartNo (none) -> CL10A475KQ8NNNC; Vendor (none) -> Digi-Key; VendorPartNo (none) -> 1276-1045-1-ND
- C17, C19, C20, C21, C22, C23, C24, C25, C26, C27, C28: Manufacturer (none) -> Samsung Electro-Mechanics; MfgPartNo (none) -> CL05A224KQ5NNNC; Vendor (none) -> Digi-Key; VendorPartNo (none) -> 1276-1124-1-ND
- C29, C30: Manufacturer (none) -> Samsung Electro-Mechanics; MfgPartNo (none) -> CL21A106KPFNNNG; Vendor (none) -> Digi-Key; VendorPartNo (none) -> 1276-6456-1-ND
