File: wifi.kicad_sch (KiCad schematic)
At the start: 1 part

Commit message: write some things down
Parts:
- U1: renamed from U?; value MCIMX6YxxVMxxxx -> MCIMX6Y2DVM09AB; Manufacturer (none) -> NXP; MfgPartNo (none) -> MCIMX6Y2DVM09AB; Vendor (none) -> Digi-Key; VendorPartNo (none) -> 568-14995-ND
Changed lines of the file:
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@@
   (symbol (lib_id "catfood:MCIMX6YxxVMxxxx") (at 60.96 60.96 0) (unit 9)
     (in_bom yes) (on_board yes) (fields_autoplaced)
-    (property "Reference" "U?" (id 0) (at 60.96 29.21 0))
-    (property "Value" "MCIMX6YxxVMxxxx" (id 1) (at 60.96 31.75 0))
+    (property "Reference" "U1" (id 0) (at 60.96 29.21 0))
+    (property "Value" "MCIMX6Y2DVM09AB" (id 1) (at 60.96 31.75 0))
     (property "Footprint" "" (id 2) (at 50.8 41.91 0)
       (effects (font (size 1.27 1.27)) hide)
@@
       (effects (font (size 1.27 1.27)) hide)
     )
+    (property "Manufacturer" "NXP" (id 4) (at 60.96 39.37 0)
+      (effects (font (size 1.27 1.27)) hide)
+    )
+    (property "MfgPartNo" "MCIMX6Y2DVM09AB" (id 5) (at 60.96 41.91 0)
+      (effects (font (size 1.27 1.27)) hide)
+    )
+    (property "Vendor" "Digi-Key" (id 6) (at 60.96 44.45 0)
+      (effects (font (size 1.27 1.27)) hide)
+    )
+    (property "VendorPartNo" "568-14995-ND" (id 7) (at 60.96 46.99 0)
+      (effects (font (size 1.27 1.27)) hide)
+    )
