File: soc_clock_ctrl.kicad_sch (KiCad schematic)
At the start: 15 parts

Commit message: Annotation
Parts:
- gave numbers to parts that had none: 15
Changed lines of the file:
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@@
   (symbol (lib_id "power:GND") (at 118.11 135.89 0) (unit 1)
     (in_bom yes) (on_board yes) (fields_autoplaced)
-    (property "Reference" "#PWR?" (id 0) (at 118.11 142.24 0)
+    (property "Reference" "#PWR0123" (id 0) (at 118.11 142.24 0)
       (effects (font (size 1.27 1.27)) hide)
     )
@@
   (symbol (lib_id "Device:Crystal_GND24_Small") (at 76.2 121.92 0) (unit 1)
     (in_bom yes) (on_board yes)
-    (property "Reference" "Y?" (id 0) (at 76.2 114.3 0))
+    (property "Reference" "Y1" (id 0) (at 76.2 114.3 0))
     (property "Value" "24MHz" (id 1) (at 76.2 116.84 0))
     (property "Footprint" "" (id 2) (at 76.2 121.92 0)
@@
   (symbol (lib_id "power:GND") (at 123.19 68.58 0) (unit 1)
     (in_bom yes) (on_board yes) (fields_autoplaced)
-    (property "Reference" "#PWR?" (id 0) (at 123.19 74.93 0)
+    (property "Reference" "#PWR0124" (id 0) (at 123.19 74.93 0)
       (effects (font (size 1.27 1.27)) hide)
     )
@@
   (symbol (lib_id "Device:C_Small") (at 67.31 129.54 0) (unit 1)
     (in_bom yes) (on_board yes) (fields_autoplaced)
-    (property "Reference" "C?" (id 0) (at 69.85 128.2762 0)
+    (property "Reference" "C92" (id 0) (at 69.85 128.2762 0)
       (effects (font (size 1.27 1.27)) (justify left))
     )
@@
   (symbol (lib_id "power:GND") (at 224.79 101.6 0) (unit 1)
     (in_bom yes) (on_board yes) (fields_autoplaced)
-    (property "Reference" "#PWR?" (id 0) (at 224.79 107.95 0)
+    (property "Reference" "#PWR0129" (id 0) (at 224.79 107.95 0)
       (effects (font (size 1.27 1.27)) hide)
     )
@@
   (symbol (lib_id "catfood:VDD_3V3") (at 184.15 74.93 0) (unit 1)
     (in_bom yes) (on_board yes) (fields_autoplaced)
-    (property "Reference" "#PWR?" (id 0) (at 184.15 78.74 0)
+    (property "Reference" "#PWR0126" (id 0) (at 184.15 78.74 0)
       (effects (font (size 1.27 1.27)) hide)
     )
@@
   (symbol (lib_id "Connector:TestPoint") (at 87.63 49.53 90) (unit 1)
     (in_bom yes) (on_board yes) (fields_autoplaced)
-    (property "Reference" "TP?" (id 0) (at 81.915 50.8001 90)
+    (property "Reference" "TP6" (id 0) (at 81.915 50.8001 90)
       (effects (font (size 1.27 1.27)) (justify left))
     )
@@
   (symbol (lib_id "power:GND") (at 224.79 88.9 0) (unit 1)
     (in_bom yes) (on_board yes) (fields_autoplaced)
-    (property "Reference" "#PWR?" (id 0) (at 224.79 95.25 0)
+    (property "Reference" "#PWR0128" (id 0) (at 224.79 95.25 0)
       (effects (font (size 1.27 1.27)) hide)
     )
@@
   (symbol (lib_id "Connector_Generic:Conn_01x03") (at 231.775 97.79 0) (unit 1)
     (in_bom yes) (on_board yes) (fields_autoplaced)
-    (property "Reference" "J?" (id 0) (at 234.95 96.5199 0)
+    (property "Reference" "J5" (id 0) (at 234.95 96.5199 0)
       (effects (font (size 1.27 1.27)) (justify left))
     )
@@
   (symbol (lib_id "power:GND") (at 109.22 68.58 0) (unit 1)
     (in_bom yes) (on_board yes) (fields_autoplaced)
-    (property "Reference" "#PWR?" (id 0) (at 109.22 74.93 0)
+    (property "Reference" "#PWR0122" (id 0) (at 109.22 74.93 0)
       (effects (font (size 1.27 1.27)) hide)
     )
@@
   (symbol (lib_id "power:GND") (at 209.55 64.77 0) (unit 1)
     (in_bom yes) (on_board yes) (fields_autoplaced)
-    (property "Reference" "#PWR?" (id 0) (at 209.55 71.12 0)
+    (property "Reference" "#PWR0127" (id 0) (at 209.55 71.12 0)
       (effects (font (size 1.27 1.27)) hide)
     )
@@
   (symbol (lib_id "catfood:MCIMX6YxxVMxxxx") (at 157.48 72.39 0) (unit 2)
     (in_bom yes) (on_board yes) (fields_autoplaced)
-    (property "Reference" "U?" (id 0) (at 154.94 43.18 0))
+    (property "Reference" "U4" (id 0) (at 154.94 43.18 0))
     (property "Value" "MCIMX6Y2DVM09AB" (id 1) (at 154.94 45.72 0))
     (property "Footprint" "" (id 2) (at 147.32 53.34 0)
@@
   (symbol (lib_id "power:GND") (at 102.87 135.89 0) (unit 1)
     (in_bom yes) (on_board yes) (fields_autoplaced)
-    (property "Reference" "#PWR?" (id 0) (at 102.87 142.24 0)
+    (property "Reference" "#PWR0121" (id 0) (at 102.87 142.24 0)
       (effects (font (size 1.27 1.27)) hide)
     )
@@
   (symbol (lib_id "Device:R_Small") (at 200.66 62.23 270) (unit 1)
     (in_bom yes) (on_board yes)
-    (property "Reference" "R?" (id 0) (at 200.66 59.69 90))
+    (property "Reference" "R46" (id 0) (at 200.66 59.69 90))
     (property "Value" "10k 0402" (id 1) (at 200.66 64.77 90))
     (property "Footprint" "" (id 2) (at 200.66 62.23 0)
@@
   (symbol (lib_id "Device:R_Small") (at 52.07 129.54 0) (unit 1)
     (in_bom yes) (on_board yes) (fields_autoplaced)
-    (property "Reference" "R?" (id 0) (at 54.61 128.2699 0)
+    (property "Reference" "R44" (id 0) (at 54.61 128.2699 0)
       (effects (font (size 1.27 1.27)) (justify left))
     )
@@
   (symbol (lib_id "Connector_Generic:Conn_01x03") (at 231.775 85.09 0) (unit 1)
     (in_bom yes) (on_board yes) (fields_autoplaced)
-    (property "Reference" "J?" (id 0) (at 234.95 83.8199 0)
+    (property "Reference" "J4" (id 0) (at 234.95 83.8199 0)
       (effects (font (size 1.27 1.27)) (justify left))
     )
@@
   (symbol (lib_id "power:GND") (at 52.07 135.89 0) (unit 1)
     (in_bom yes) (on_board yes) (fields_autoplaced)
-    (property "Reference" "#PWR?" (id 0) (at 52.07 142.24 0)
+    (property "Reference" "#PWR0117" (id 0) (at 52.07 142.24 0)
       (effects (font (size 1.27 1.27)) hide)
     )
@@
   (symbol (lib_id "Device:C_Small") (at 118.11 129.54 0) (unit 1)
     (in_bom yes) (on_board yes) (fields_autoplaced)
-    (property "Reference" "C?" (id 0) (at 120.65 128.2762 0)
+    (property "Reference" "C95" (id 0) (at 120.65 128.2762 0)
       (effects (font (size 1.27 1.27)) (justify left))
     )
@@
   (symbol (lib_id "Device:C_Small") (at 82.55 129.54 0) (unit 1)
     (in_bom yes) (on_board yes) (fields_autoplaced)
-    (property "Reference" "C?" (id 0) (at 85.09 128.2762 0)
+    (property "Reference" "C93" (id 0) (at 85.09 128.2762 0)
       (effects (font (size 1.27 1.27)) (justify left))
     )
@@
   (symbol (lib_id "catfood:VDD_3V3_IN") (at 91.44 58.42 0) (unit 1)
     (in_bom yes) (on_board yes)
-    (property "Reference" "#PWR?" (id 0) (at 91.44 62.23 0)
+    (property "Reference" "#PWR0120" (id 0) (at 91.44 62.23 0)
       (effects (font (size 1.27 1.27)) hide)
     )
@@
   (symbol (lib_id "Device:Crystal_Small") (at 110.49 124.46 0) (unit 1)
     (in_bom yes) (on_board yes) (fields_autoplaced)
-    (property "Reference" "Y?" (id 0) (at 110.49 118.11 0))
+    (property "Reference" "Y2" (id 0) (at 110.49 118.11 0))
     (property "Value" "32.768kHz" (id 1) (at 110.49 120.65 0))
     (property "Footprint" "" (id 2) (at 110.49 124.46 0)
@@
   (symbol (lib_id "power:GND") (at 82.55 135.89 0) (unit 1)
     (in_bom yes) (on_board yes) (fields_autoplaced)
-    (property "Reference" "#PWR?" (id 0) (at 82.55 142.24 0)
+    (property "Reference" "#PWR0119" (id 0) (at 82.55 142.24 0)
       (effects (font (size 1.27 1.27)) hide)
     )
@@
   (symbol (lib_id "Connector:TestPoint") (at 87.63 52.07 90) (unit 1)
     (in_bom yes) (on_board yes) (fields_autoplaced)
-    (property "Reference" "TP?" (id 0) (at 81.915 53.3401 90)
+    (property "Reference" "TP7" (id 0) (at 81.915 53.3401 90)
       (effects (font (size 1.27 1.27)) (justify left))
     )
@@
   (symbol (lib_id "Device:C_Small") (at 102.87 129.54 0) (unit 1)
     (in_bom yes) (on_board yes) (fields_autoplaced)
-    (property "Reference" "C?" (id 0) (at 105.41 128.2762 0)
+    (property "Reference" "C94" (id 0) (at 105.41 128.2762 0)
       (effects (font (size 1.27 1.27)) (justify left))
     )
@@
   (symbol (lib_id "Jumper:SolderJumper_2_Open") (at 100.33 59.69 0) (unit 1)
     (in_bom yes) (on_board yes)
-    (property "Reference" "JP?" (id 0) (at 100.33 57.15 0))
+    (property "Reference" "JP1" (id 0) (at 100.33 57.15 0))
     (property "Value" "SolderJumper_2_Open" (id 1) (at 100.33 55.88 0)
       (effects (font (size 1.27 1.27)) hide)
@@
   (symbol (lib_id "power:GND") (at 67.31 135.89 0) (unit 1)
     (in_bom yes) (on_board yes) (fields_autoplaced)
-    (property "Reference" "#PWR?" (id 0) (at 67.31 142.24 0)
+    (property "Reference" "#PWR0118" (id 0) (at 67.31 142.24 0)
       (effects (font (size 1.27 1.27)) hide)
     )
@@
   (symbol (lib_id "Device:R_Small") (at 109.22 63.5 0) (unit 1)
     (in_bom yes) (on_board yes) (fields_autoplaced)
-    (property "Reference" "R?" (id 0) (at 111.76 62.2299 0)
+    (property "Reference" "R45" (id 0) (at 111.76 62.2299 0)
       (effects (font (size 1.27 1.27)) (justify left))
     )
@@
   (symbol (lib_id "power:GND") (at 128.27 68.58 0) (unit 1)
     (in_bom yes) (on_board yes) (fields_autoplaced)
-    (property "Reference" "#PWR?" (id 0) (at 128.27 74.93 0)
-      (effects (font (size 1.27 1.27)) hide)
-    )
+    (property "Reference" "#PWR0125" (id 0) (at 128.27 74.93 0)
+      (effects (font (size 1.27 1.27)) hide)
+    )
