File: soc_clock_ctrl.kicad_sch (KiCad schematic)
At the start: 15 parts, among them J4 Conn_01x03, J5 Conn_01x03, U4 MCIMX6Y2DVM09AB, Y1 24MHz, Y2 32.768kHz

Commit message: Footprint assignments for standard passives
Parts:
- C92, C93, C94, C95: footprint (none) -> Capacitor_SMD:C_0402_1005Metric
- J4, J5: footprint (none) -> Connector_PinHeader_1.27mm:PinHeader_1x03_P1.27mm_Vertical_SMD_Pin1Left
- R44, R45, R46: footprint (none) -> Resistor_SMD:R_0402_1005Metric
- TP6, TP7: footprint (none) -> TestPoint:TestPoint_Pad_D1.5mm
Changed lines of the file:
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@@
       (effects (font (size 1.27 1.27)) (justify left))
     )
-    (property "Footprint" "" (id 2) (at 67.31 129.54 0)
+    (property "Footprint" "Capacitor_SMD:C_0402_1005Metric" (id 2) (at 67.31 129.54 0)
       (effects (font (size 1.27 1.27)) hide)
     )
@@
       (effects (font (size 1.27 1.27)) (justify left) hide)
     )
-    (property "Footprint" "" (id 2) (at 87.63 44.45 0)
+    (property "Footprint" "TestPoint:TestPoint_Pad_D1.5mm" (id 2) (at 87.63 44.45 0)
       (effects (font (size 1.27 1.27)) hide)
     )
@@
       (effects (font (size 1.27 1.27)) (justify left))
     )
-    (property "Footprint" "" (id 2) (at 231.775 97.79 0)
+    (property "Footprint" "Connector_PinHeader_1.27mm:PinHeader_1x03_P1.27mm_Vertical_SMD_Pin1Left" (id 2) (at 231.775 97.79 0)
       (effects (font (size 1.27 1.27)) hide)
     )
@@
     (property "Reference" "R46" (id 0) (at 200.66 59.69 90))
     (property "Value" "10k 0402" (id 1) (at 200.66 64.77 90))
-    (property "Footprint" "" (id 2) (at 200.66 62.23 0)
+    (property "Footprint" "Resistor_SMD:R_0402_1005Metric" (id 2) (at 200.66 62.23 0)
       (effects (font (size 1.27 1.27)) hide)
     )
@@
       (effects (font (size 1.27 1.27)) (justify left))
     )
-    (property "Footprint" "" (id 2) (at 52.07 129.54 0)
+    (property "Footprint" "Resistor_SMD:R_0402_1005Metric" (id 2) (at 52.07 129.54 0)
       (effects (font (size 1.27 1.27)) hide)
     )
@@
       (effects (font (size 1.27 1.27)) (justify left))
     )
-    (property "Footprint" "" (id 2) (at 231.775 85.09 0)
+    (property "Footprint" "Connector_PinHeader_1.27mm:PinHeader_1x03_P1.27mm_Vertical_SMD_Pin1Left" (id 2) (at 231.775 85.09 0)
       (effects (font (size 1.27 1.27)) hide)
     )
@@
       (effects (font (size 1.27 1.27)) (justify left))
     )
-    (property "Footprint" "" (id 2) (at 118.11 129.54 0)
+    (property "Footprint" "Capacitor_SMD:C_0402_1005Metric" (id 2) (at 118.11 129.54 0)
       (effects (font (size 1.27 1.27)) hide)
     )
@@
       (effects (font (size 1.27 1.27)) (justify left))
     )
-    (property "Footprint" "" (id 2) (at 82.55 129.54 0)
+    (property "Footprint" "Capacitor_SMD:C_0402_1005Metric" (id 2) (at 82.55 129.54 0)
       (effects (font (size 1.27 1.27)) hide)
     )
@@
       (effects (font (size 1.27 1.27)) (justify left) hide)
     )
-    (property "Footprint" "" (id 2) (at 87.63 46.99 0)
+    (property "Footprint" "TestPoint:TestPoint_Pad_D1.5mm" (id 2) (at 87.63 46.99 0)
       (effects (font (size 1.27 1.27)) hide)
     )
@@
       (effects (font (size 1.27 1.27)) (justify left))
     )
-    (property "Footprint" "" (id 2) (at 102.87 129.54 0)
+    (property "Footprint" "Capacitor_SMD:C_0402_1005Metric" (id 2) (at 102.87 129.54 0)
       (effects (font (size 1.27 1.27)) hide)
     )
@@
       (effects (font (size 1.27 1.27)) (justify left))
     )
-    (property "Footprint" "" (id 2) (at 109.22 63.5 0)
-      (effects (font (size 1.27 1.27)) hide)
-    )
+    (property "Footprint" "Resistor_SMD:R_0402_1005Metric" (id 2) (at 109.22 63.5 0)
+      (effects (font (size 1.27 1.27)) hide)
+    )
