File: gpio.kicad_sch (KiCad schematic)
At the start: 7 parts, among them U4 MCIMX6Y2DVM09AB

Commit message: Footprint assignments for standard passives
Parts:
- C86, C87, C88, C89, C90, C91: footprint (none) -> Capacitor_SMD:C_0402_1005Metric
Changed lines of the file:
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@@
       (effects (font (size 1.27 1.27)) (justify left))
     )
-    (property "Footprint" "" (id 2) (at 136.525 96.52 0)
+    (property "Footprint" "Capacitor_SMD:C_0402_1005Metric" (id 2) (at 136.525 96.52 0)
       (effects (font (size 1.27 1.27)) hide)
     )
@@
       (effects (font (size 1.27 1.27)) (justify left))
     )
-    (property "Footprint" "" (id 2) (at 19.05 42.545 0)
+    (property "Footprint" "Capacitor_SMD:C_0402_1005Metric" (id 2) (at 19.05 42.545 0)
       (effects (font (size 1.27 1.27)) hide)
     )
@@
       (effects (font (size 1.27 1.27)) (justify left))
     )
-    (property "Footprint" "" (id 2) (at 153.67 96.52 0)
+    (property "Footprint" "Capacitor_SMD:C_0402_1005Metric" (id 2) (at 153.67 96.52 0)
       (effects (font (size 1.27 1.27)) hide)
     )
@@
       (effects (font (size 1.27 1.27)) (justify left))
     )
-    (property "Footprint" "" (id 2) (at 24.13 144.78 0)
+    (property "Footprint" "Capacitor_SMD:C_0402_1005Metric" (id 2) (at 24.13 144.78 0)
       (effects (font (size 1.27 1.27)) hide)
     )
@@
       (effects (font (size 1.27 1.27)) (justify left))
     )
-    (property "Footprint" "" (id 2) (at 168.91 41.91 0)
+    (property "Footprint" "Capacitor_SMD:C_0402_1005Metric" (id 2) (at 168.91 41.91 0)
       (effects (font (size 1.27 1.27)) hide)
     )
@@
       (effects (font (size 1.27 1.27)) (justify left))
     )
-    (property "Footprint" "" (id 2) (at 163.83 140.335 0)
-      (effects (font (size 1.27 1.27)) hide)
-    )
+    (property "Footprint" "Capacitor_SMD:C_0402_1005Metric" (id 2) (at 163.83 140.335 0)
+      (effects (font (size 1.27 1.27)) hide)
+    )
