File: gpio.kicad_sch (KiCad schematic)
At the start: 7 parts, among them U4 MCIMX6Y2DVM09AB

Commit message: Update fields
Parts:
- C86, C87, C89, C90, C91: Manufacturer (none) -> Samsung Electro-Mechanics; MfgPartNo (none) -> CL05A224KQ5NNNC; Vendor (none) -> Digi-Key; VendorPartNo (none) -> 1276-1124-1-ND
- C88: Manufacturer (none) -> TDK Corporation; MfgPartNo (none) -> CGB2A1X5R1E105K033BC; Vendor (none) -> Digi-Key; VendorPartNo (none) -> 445-13185-1-ND
Changed lines of the file:
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@@
 )
         (pin "2"
-))
+)
+        (property "Manufacturer" "TDK Corporation"
+            (id 4)
+            (at 139.7 105.4162 0)
+            (effects
+                (font
+                    (size 1.27 1.27))
+                (justify left) hide))
+        (property "MfgPartNo" "CGB2A1X5R1E105K033BC"
+            (id 5)
+            (at 139.7 107.95620000000001 0)
+            (effects
+                (font
+                    (size 1.27 1.27))
+                (justify left) hide))
+        (property "Vendor" "Digi-Key"
+            (id 6)
+            (at 139.7 110.4962 0)
+            (effects
+                (font
+                    (size 1.27 1.27))
+                (justify left) hide))
+        (property "VendorPartNo" "445-13185-1-ND"
+            (id 7)
+            (at 139.7 113.03620000000001 0)
+            (effects
+                (font
+                    (size 1.27 1.27))
+                (justify left) hide)))
     (symbol
         (lib_id "power:GND")
@@
                 (font
                     (size 1.27 1.27)) hide))
-        (property "Datasheet" ""
+        (property "Datasheet" "~"
             (id 3)
             (at 195.58 39.37 0)
@@
                 (font
                     (size 1.27 1.27)) hide))
-        (property "Datasheet" ""
+        (property "Datasheet" "~"
             (id 3)
             (at 189.865 139.065 0)
@@
 )
         (pin "2"
-))
+)
+        (property "Manufacturer" "Samsung Electro-Mechanics"
+            (id 4)
+            (at 21.59 51.441199999999995 0)
+            (effects
+                (font
+                    (size 1.27 1.27))
+                (justify left) hide))
+        (property "MfgPartNo" "CL05A224KQ5NNNC"
+            (id 5)
+            (at 21.59 53.9812 0)
+            (effects
+                (font
+                    (size 1.27 1.27))
+                (justify left) hide))
+        (property "Vendor" "Digi-Key"
+            (id 6)
+            (at 21.59 56.5212 0)
+            (effects
+                (font
+                    (size 1.27 1.27))
+                (justify left) hide))
+        (property "VendorPartNo" "1276-1124-1-ND"
+            (id 7)
+            (at 21.59 59.0612 0)
+            (effects
+                (font
+                    (size 1.27 1.27))
+                (justify left) hide)))
     (symbol
         (lib_name "MCIMX6YxxVMxxxx_1")
@@
                 (font
                     (size 1.27 1.27)) hide))
-        (property "Datasheet" ""
+        (property "Datasheet" "~"
             (id 3)
             (at 50.165 142.875 0)
@@
 )
         (pin "2"
-))
+)
+        (property "Manufacturer" "Samsung Electro-Mechanics"
+            (id 4)
+            (at 156.21 105.4162 0)
+            (effects
+                (font
+                    (size 1.27 1.27))
+                (justify left) hide))
+        (property "MfgPartNo" "CL05A224KQ5NNNC"
+            (id 5)
+            (at 156.21 107.95620000000001 0)
+            (effects
+                (font
+                    (size 1.27 1.27))
+                (justify left) hide))
+        (property "Vendor" "Digi-Key"
+            (id 6)
+            (at 156.21 110.4962 0)
+            (effects
+                (font
+                    (size 1.27 1.27))
+                (justify left) hide))
+        (property "VendorPartNo" "1276-1124-1-ND"
+            (id 7)
+            (at 156.21 113.03620000000001 0)
+            (effects
+                (font
+                    (size 1.27 1.27))
+                (justify left) hide)))
     (symbol
         (lib_id "Device:C_Small")
@@
 )
         (pin "2"
-))
+)
+        (property "Manufacturer" "Samsung Electro-Mechanics"
+            (id 4)
+            (at 26.67 153.6762 0)
+            (effects
+                (font
+                    (size 1.27 1.27))
+                (justify left) hide))
+        (property "MfgPartNo" "CL05A224KQ5NNNC"
+            (id 5)
+            (at 26.67 156.2162 0)
+            (effects
+                (font
+                    (size 1.27 1.27))
+                (justify left) hide))
+        (property "Vendor" "Digi-Key"
+            (id 6)
+            (at 26.67 158.7562 0)
+            (effects
+                (font
+                    (size 1.27 1.27))
+                (justify left) hide))
+        (property "VendorPartNo" "1276-1124-1-ND"
+            (id 7)
+            (at 26.67 161.2962 0)
+            (effects
+                (font
+                    (size 1.27 1.27))
+                (justify left) hide)))
     (symbol
         (lib_name "MCIMX6YxxVMxxxx_2")
@@
                 (font
                     (size 1.27 1.27)) hide))
-        (property "Datasheet" ""
+        (property "Datasheet" "~"
             (id 3)
             (at 44.45 40.64 0)
@@
                 (font
                     (size 1.27 1.27)) hide))
-        (property "Datasheet" ""
+        (property "Datasheet" "~"
             (id 3)
             (at 182.88 95.25 0)
@@
 )
         (pin "2"
-))
+)
+        (property "Manufacturer" "Samsung Electro-Mechanics"
+            (id 4)
+            (at 171.45 50.806200000000004 0)
+            (effects
+                (font
+                    (size 1.27 1.27))
+                (justify left) hide))
+        (property "MfgPartNo" "CL05A224KQ5NNNC"
+            (id 5)
+            (at 171.45 53.346199999999996 0)
+            (effects
+                (font
+                    (size 1.27 1.27))
+                (justify left) hide))
+        (property "Vendor" "Digi-Key"
+            (id 6)
+            (at 171.45 55.8862 0)
+            (effects
+                (font
+                    (size 1.27 1.27))
+                (justify left) hide))
+        (property "VendorPartNo" "1276-1124-1-ND"
+            (id 7)
+            (at 171.45 58.4262 0)
+            (effects
+                (font
+                    (size 1.27 1.27))
+                (justify left) hide)))
     (symbol
         (lib_id "catfood:VDD_3V3")
@@
 )
         (pin "2"
-))
+)
+        (property "Manufacturer" "Samsung Electro-Mechanics"
+            (id 4)
+            (at 166.37 149.2312 0)
+            (effects
+                (font
+                    (size 1.27 1.27))
+                (justify left) hide))
+        (property "MfgPartNo" "CL05A224KQ5NNNC"
+            (id 5)
+            (at 166.37 151.7712 0)
+            (effects
+                (font
+                    (size 1.27 1.27))
+                (justify left) hide))
+        (property "Vendor" "Digi-Key"
+            (id 6)
+            (at 166.37 154.3112 0)
+            (effects
+                (font
+                    (size 1.27 1.27))
+                (justify left) hide))
+        (property "VendorPartNo" "1276-1124-1-ND"
+            (id 7)
+            (at 166.37 156.8512 0)
+            (effects
+                (font
+                    (size 1.27 1.27))
+                (justify left) hide)))
     (symbol
         (lib_id "catfood:VDD_3V3")
