File: usb.kicad_sch (KiCad schematic)
At the start: 22 parts, among them J1 USB4110, J2 USB_A, U4 MCIMX6Y2DVM09AB, U5 AP22615AWU-7

Commit message: ERC: power flags
Changed lines of the file:
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@@
   (junction (at 207.645 92.71) (diameter 0) (color 0 0 0 0)
+  )
+  (junction (at 55.245 151.13) (diameter 0) (color 0 0 0 0)
   )
   (junction (at 31.75 191.77) (diameter 0) (color 0 0 0 0)
@@
     (stroke (width 0) (type default) (color 0 0 0 0))
   )
-  (wire (pts (xy 46.99 151.13) (xy 103.505 151.13))
+  (wire (pts (xy 46.99 151.13) (xy 55.245 151.13))
     (stroke (width 0) (type default) (color 0 0 0 0))
   )
@@
     (stroke (width 0) (type default) (color 0 0 0 0))
   )
+  (wire (pts (xy 55.245 151.13) (xy 103.505 151.13))
+    (stroke (width 0) (type default) (color 0 0 0 0))
+  )
   (wire (pts (xy 91.44 39.37) (xy 91.44 43.18))
     (stroke (width 0) (type default) (color 0 0 0 0))
@@
     (stroke (width 0) (type default) (color 0 0 0 0))
   )
+  (wire (pts (xy 38.735 190.5) (xy 38.735 191.77))
+    (stroke (width 0) (type default) (color 0 0 0 0))
+  )
   (wire (pts (xy 48.895 163.83) (xy 48.895 166.37))
     (stroke (width 0) (type default) (color 0 0 0 0))
@@
     (stroke (width 0) (type default) (color 0 0 0 0))
   )
+  (wire (pts (xy 55.245 149.225) (xy 55.245 151.13))
+    (stroke (width 0) (type default) (color 0 0 0 0))
+  )
   (wire (pts (xy 229.87 125.095) (xy 229.87 127.635))
     (stroke (width 0) (type default) (color 0 0 0 0))
@@
   )
   (wire (pts (xy 46.99 158.75) (xy 57.785 158.75))
+    (stroke (width 0) (type default) (color 0 0 0 0))
+  )
+  (wire (pts (xy 38.735 191.77) (xy 31.75 191.77))
     (stroke (width 0) (type default) (color 0 0 0 0))
   )
@@
     (pin "1")
     (pin "2")
+  )
+  (symbol (lib_id "power:PWR_FLAG") (at 38.735 190.5 0) (unit 1)
+    (in_bom yes) (on_board yes) (fields_autoplaced)
+    (property "Reference" "#FLG01" (id 0) (at 38.735 188.595 0)
+      (effects (font (size 1.27 1.27)) hide)
+    )
+    (property "Value" "PWR_FLAG" (id 1) (at 38.735 185.42 0))
+    (property "Footprint" "" (id 2) (at 38.735 190.5 0)
+      (effects (font (size 1.27 1.27)) hide)
+    )
+    (property "Datasheet" "~" (id 3) (at 38.735 190.5 0)
+      (effects (font (size 1.27 1.27)) hide)
+    )
+    (pin "1")
   )
   (symbol (lib_id "power:GND") (at 116.205 115.57 0) (unit 1)
@@
       (effects (font (size 1.27 1.27)) hide)
     )
+    (pin "1")
+  )
+  (symbol (lib_id "power:PWR_FLAG") (at 55.245 149.225 0) (unit 1)
+    (in_bom yes) (on_board yes) (fields_autoplaced)
+    (property "Reference" "#FLG02" (id 0) (at 55.245 147.32 0)
+      (effects (font (size 1.27 1.27)) hide)
+    )
+    (property "Value" "PWR_FLAG" (id 1) (at 55.245 144.145 0))
+    (property "Footprint" "" (id 2) (at 55.245 149.225 0)
+      (effects (font (size 1.27 1.27)) hide)
+    )
+    (property "Datasheet" "~" (id 3) (at 55.245 149.225 0)
+      (effects (font (size 1.27 1.27)) hide)
+    )

Commit message: Update symbols
Connections:
- net USB_OTG2_VBUS: now also U5.1 (VOUT); no longer U5. (VOUT)
Changed lines of the file:
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@@
       (effects (font (size 1.27 1.27)) hide)
     )
-    (pin "")
+    (pin "1")
     (pin "2")
     (pin "3")

Commit message: BOM consolidation
Parts:
- C35, C36: value 1uF 0603 -> 1uF 0402
Changed lines of the file:
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@@
       (effects (font (size 1.27 1.27)) (justify left))
     )
-    (property "Value" "1uF 0603" (id 1) (at 73.66 55.2512 0)
+    (property "Value" "1uF 0402" (id 1) (at 73.66 55.2512 0)
       (effects (font (size 1.27 1.27)) (justify left))
     )
@@
   (symbol (lib_id "Device:C_Small") (at 91.44 36.83 0) (unit 1)
     (in_bom yes) (on_board yes) (fields_autoplaced)
-    (property "Reference" "C36" (id 0) (at 94.615 35.5662 0)
-      (effects (font (size 1.27 1.27)) (justify left))
-    )
-    (property "Value" "1uF 0603" (id 1) (at 94.615 38.1062 0)
-      (effects (font (size 1.27 1.27)) (justify left))
-    )
+    (property "Reference" "C36" (id 0) (at 93.98 35.5662 0)
+      (effects (font (size 1.27 1.27)) (justify left))
+    )
+    (property "Value" "1uF 0402" (id 1) (at 93.98 38.1062 0)
+      (effects (font (size 1.27 1.27)) (justify left))
+    )

Commit message: Footprint assignments for standard passives
Parts:
- C33, C38, C39, C41: footprint (none) -> Capacitor_SMD:C_0805_2012Metric
- C34, C35, C36, C37, C42: footprint (none) -> Capacitor_SMD:C_0402_1005Metric
- C40: footprint (none) -> Capacitor_SMD:C_1210_3225Metric
- D2, D5: footprint Package_TO_SOT_SMD:SOT-416 -> (none)
- D3, D4: footprint Diode_SMD:D_SMF -> (none)
- R10, R11, R12, R9: footprint (none) -> Resistor_SMD:R_0402_1005Metric
Changed lines of the file:
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@@
       (effects (font (size 1.27 1.27)) (justify left))
     )
-    (property "Footprint" "" (id 2) (at 71.755 97.79 0)
+    (property "Footprint" "Resistor_SMD:R_0402_1005Metric" (id 2) (at 71.755 97.79 0)
       (effects (font (size 1.27 1.27)) hide)
     )
@@
       (effects (font (size 0.8 0.8)))
     )
-    (property "Footprint" "" (id 2) (at 60.325 158.75 0)
+    (property "Footprint" "Resistor_SMD:R_0402_1005Metric" (id 2) (at 60.325 158.75 0)
       (effects (font (size 1.27 1.27)) hide)
     )
@@
       (effects (font (size 1.27 1.27)) (justify left))
     )
-    (property "Footprint" "" (id 2) (at 70.485 53.975 0)
+    (property "Footprint" "Capacitor_SMD:C_0402_1005Metric" (id 2) (at 70.485 53.975 0)
       (effects (font (size 1.27 1.27)) hide)
     )
@@
       (effects (font (size 1.27 1.27)) (justify left))
     )
-    (property "Footprint" "" (id 2) (at 46.355 96.52 0)
+    (property "Footprint" "Capacitor_SMD:C_0402_1005Metric" (id 2) (at 46.355 96.52 0)
       (effects (font (size 1.27 1.27)) hide)
     )
@@
       (effects (font (size 1.27 1.27)) (justify left))
     )
-    (property "Footprint" "" (id 2) (at 141.605 97.79 0)
+    (property "Footprint" "Capacitor_SMD:C_0805_2012Metric" (id 2) (at 141.605 97.79 0)
       (effects (font (size 1.27 1.27)) hide)
     )
@@
       (effects (font (size 1.27 1.27)) (justify left))
     )
-    (property "Footprint" "" (id 2) (at 157.48 97.79 0)
+    (property "Footprint" "Capacitor_SMD:C_0805_2012Metric" (id 2) (at 157.48 97.79 0)
       (effects (font (size 1.27 1.27)) hide)
     )
@@
       (effects (font (size 1.27 1.27)) (justify left))
     )
-    (property "Footprint" "Diode_SMD:D_SMF" (id 2) (at 207.645 118.745 0)
+    (property "Footprint" "" (id 2) (at 207.645 118.745 0)
       (effects (font (size 1.27 1.27)) hide)
     )
@@
       (effects (font (size 1.27 1.27)) (justify right))
     )
-    (property "Footprint" "Package_TO_SOT_SMD:SOT-416" (id 2) (at 237.49 120.015 0)
+    (property "Footprint" "" (id 2) (at 237.49 120.015 0)
       (effects (font (size 1.27 1.27)) hide)
     )
@@
       (effects (font (size 1.27 1.27)) (justify right))
     )
-    (property "Footprint" "Package_TO_SOT_SMD:SOT-416" (id 2) (at 75.565 179.705 0)
+    (property "Footprint" "" (id 2) (at 75.565 179.705 0)
       (effects (font (size 1.27 1.27)) hide)
     )
@@
       (effects (font (size 1.27 1.27)) (justify left))
     )
-    (property "Footprint" "" (id 2) (at 125.095 97.79 0)
+    (property "Footprint" "Capacitor_SMD:C_0402_1005Metric" (id 2) (at 125.095 97.79 0)
       (effects (font (size 1.27 1.27)) hide)
     )
@@
       (effects (font (size 1.27 1.27)) (justify left))
     )
-    (property "Footprint" "Diode_SMD:D_SMF" (id 2) (at 103.505 159.385 0)
+    (property "Footprint" "" (id 2) (at 103.505 159.385 0)
       (effects (font (size 1.27 1.27)) hide)
     )
@@
       (effects (font (size 1.27 1.27)) (justify left))
     )
-    (property "Footprint" "" (id 2) (at 179.07 48.26 0)
+    (property "Footprint" "Capacitor_SMD:C_0805_2012Metric" (id 2) (at 179.07 48.26 0)
       (effects (font (size 1.27 1.27)) hide)
     )
@@
       (effects (font (size 1.27 1.27)) (justify left))
     )
-    (property "Footprint" "" (id 2) (at 91.44 36.83 0)
+    (property "Footprint" "Capacitor_SMD:C_0402_1005Metric" (id 2) (at 91.44 36.83 0)
       (effects (font (size 1.27 1.27)) hide)
     )
@@
       (effects (font (size 1.27 1.27)) (justify left))
     )
-    (property "Footprint" "" (id 2) (at 116.205 110.49 0)
+    (property "Footprint" "Resistor_SMD:R_0402_1005Metric" (id 2) (at 116.205 110.49 0)
       (effects (font (size 1.27 1.27)) hide)
     )
@@
       (effects (font (size 1.27 1.27)) (justify left))
     )
-    (property "Footprint" "" (id 2) (at 29.845 96.52 0)
+    (property "Footprint" "Capacitor_SMD:C_0805_2012Metric" (id 2) (at 29.845 96.52 0)
       (effects (font (size 1.27 1.27)) hide)
     )
@@
       (effects (font (size 1.27 1.27)) (justify left))
     )
-    (property "Footprint" "" (id 2) (at 172.72 97.79 0)
+    (property "Footprint" "Capacitor_SMD:C_1210_3225Metric" (id 2) (at 172.72 97.79 0)
       (effects (font (size 1.27 1.27)) hide)
     )
@@
       (effects (font (size 1.27 1.27)) (justify left))
     )
-    (property "Footprint" "" (id 2) (at 194.945 48.26 0)
+    (property "Footprint" "Capacitor_SMD:C_0402_1005Metric" (id 2) (at 194.945 48.26 0)
       (effects (font (size 1.27 1.27)) hide)
     )
@@
       (effects (font (size 0.8 0.8)))
     )
-    (property "Footprint" "" (id 2) (at 60.325 156.21 0)
-      (effects (font (size 1.27 1.27)) hide)
-    )
+    (property "Footprint" "Resistor_SMD:R_0402_1005Metric" (id 2) (at 60.325 156.21 0)
+      (effects (font (size 1.27 1.27)) hide)
+    )
