File: catfood.kicad_sch (KiCad schematic)
At the start: 8 parts

Commit message: Update fields
Parts:
- H1, H2, H3, H4, H5, H6, H7, H8: Manufacturer (none) -> N/A; MfgPartNo (none) -> N/A; Vendor (none) -> N/A; VendorPartNo (none) -> N/A
Changed lines of the file:
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@@
             (effects
                 (font
-                    (size 1.27 1.27)) hide)))
+                    (size 1.27 1.27)) hide))
+        (property "Manufacturer" "N/A"
+            (id 4)
+            (at 220.345 83.81989999999999 0)
+            (effects
+                (font
+                    (size 1.27 1.27))
+                (justify left) hide))
+        (property "MfgPartNo" "N/A"
+            (id 5)
+            (at 220.345 86.3599 0)
+            (effects
+                (font
+                    (size 1.27 1.27))
+                (justify left) hide))
+        (property "Vendor" "N/A"
+            (id 6)
+            (at 220.345 88.89989999999999 0)
+            (effects
+                (font
+                    (size 1.27 1.27))
+                (justify left) hide))
+        (property "VendorPartNo" "N/A"
+            (id 7)
+            (at 220.345 91.4399 0)
+            (effects
+                (font
+                    (size 1.27 1.27))
+                (justify left) hide)))
     (symbol
         (lib_id "power:GND")
@@
                     (size 1.27 1.27)) hide))
         (pin "1"
-))
+)
+        (property "Manufacturer" "N/A"
+            (id 4)
+            (at 182.245 93.3449 0)
+            (effects
+                (font
+                    (size 1.27 1.27))
+                (justify left) hide))
+        (property "MfgPartNo" "N/A"
+            (id 5)
+            (at 182.245 95.8849 0)
+            (effects
+                (font
+                    (size 1.27 1.27))
+                (justify left) hide))
+        (property "Vendor" "N/A"
+            (id 6)
+            (at 182.245 98.4249 0)
+            (effects
+                (font
+                    (size 1.27 1.27))
+                (justify left) hide))
+        (property "VendorPartNo" "N/A"
+            (id 7)
+            (at 182.245 100.9649 0)
+            (effects
+                (font
+                    (size 1.27 1.27))
+                (justify left) hide)))
     (symbol
         (lib_id "power:GND")
@@
                     (size 1.27 1.27)) hide))
         (pin "1"
-))
+)
+        (property "Manufacturer" "N/A"
+            (id 4)
+            (at 182.245 76.83489999999999 0)
+            (effects
+                (font
+                    (size 1.27 1.27))
+                (justify left) hide))
+        (property "MfgPartNo" "N/A"
+            (id 5)
+            (at 182.245 79.3749 0)
+            (effects
+                (font
+                    (size 1.27 1.27))
+                (justify left) hide))
+        (property "Vendor" "N/A"
+            (id 6)
+            (at 182.245 81.91489999999999 0)
+            (effects
+                (font
+                    (size 1.27 1.27))
+                (justify left) hide))
+        (property "VendorPartNo" "N/A"
+            (id 7)
+            (at 182.245 84.4549 0)
+            (effects
+                (font
+                    (size 1.27 1.27))
+                (justify left) hide)))
     (symbol
         (lib_id "Mechanical:MountingHole")
@@
             (effects
                 (font
-                    (size 1.27 1.27)) hide)))
+                    (size 1.27 1.27)) hide))
+        (property "Manufacturer" "N/A"
+            (id 4)
+            (at 220.345 96.51989999999999 0)
+            (effects
+                (font
+                    (size 1.27 1.27))
+                (justify left) hide))
+        (property "MfgPartNo" "N/A"
+            (id 5)
+            (at 220.345 99.0599 0)
+            (effects
+                (font
+                    (size 1.27 1.27))
+                (justify left) hide))
+        (property "Vendor" "N/A"
+            (id 6)
+            (at 220.345 101.59989999999999 0)
+            (effects
+                (font
+                    (size 1.27 1.27))
+                (justify left) hide))
+        (property "VendorPartNo" "N/A"
+            (id 7)
+            (at 220.345 104.1399 0)
+            (effects
+                (font
+                    (size 1.27 1.27))
+                (justify left) hide)))
     (symbol
         (lib_id "Mechanical:MountingHole")
@@
             (effects
                 (font
-                    (size 1.27 1.27)) hide)))
+                    (size 1.27 1.27)) hide))
+        (property "Manufacturer" "N/A"
+            (id 4)
+            (at 220.345 77.4699 0)
+            (effects
+                (font
+                    (size 1.27 1.27))
+                (justify left) hide))
+        (property "MfgPartNo" "N/A"
+            (id 5)
+            (at 220.345 80.0099 0)
+            (effects
+                (font
+                    (size 1.27 1.27))
+                (justify left) hide))
+        (property "Vendor" "N/A"
+            (id 6)
+            (at 220.345 82.5499 0)
+            (effects
+                (font
+                    (size 1.27 1.27))
+                (justify left) hide))
+        (property "VendorPartNo" "N/A"
+            (id 7)
+            (at 220.345 85.0899 0)
+            (effects
+                (font
+                    (size 1.27 1.27))
+                (justify left) hide)))
     (symbol
         (lib_id "power:GND")
@@
                     (size 1.27 1.27)) hide))
         (pin "1"
-))
+)
+        (property "Manufacturer" "N/A"
+            (id 4)
+            (at 192.405 93.3449 0)
+            (effects
+                (font
+                    (size 1.27 1.27))
+                (justify left) hide))
+        (property "MfgPartNo" "N/A"
+            (id 5)
+            (at 192.405 95.8849 0)
+            (effects
+                (font
+                    (size 1.27 1.27))
+                (justify left) hide))
+        (property "Vendor" "N/A"
+            (id 6)
+            (at 192.405 98.4249 0)
+            (effects
+                (font
+                    (size 1.27 1.27))
+                (justify left) hide))
+        (property "VendorPartNo" "N/A"
+            (id 7)
+            (at 192.405 100.9649 0)
+            (effects
+                (font
+                    (size 1.27 1.27))
+                (justify left) hide)))
     (symbol
         (lib_id "Mechanical:MountingHole_Pad")
@@
                     (size 1.27 1.27)) hide))
         (pin "1"
-))
+)
+        (property "Manufacturer" "N/A"
+            (id 4)
+            (at 192.405 76.83489999999999 0)
+            (effects
+                (font
+                    (size 1.27 1.27))
+                (justify left) hide))
+        (property "MfgPartNo" "N/A"
+            (id 5)
+            (at 192.405 79.3749 0)
+            (effects
+                (font
+                    (size 1.27 1.27))
+                (justify left) hide))
+        (property "Vendor" "N/A"
+            (id 6)
+            (at 192.405 81.91489999999999 0)
+            (effects
+                (font
+                    (size 1.27 1.27))
+                (justify left) hide))
+        (property "VendorPartNo" "N/A"
+            (id 7)
+            (at 192.405 84.4549 0)
+            (effects
+                (font
+                    (size 1.27 1.27))
+                (justify left) hide)))
     (symbol
         (lib_id "Mechanical:MountingHole")
@@
             (effects
                 (font
-                    (size 1.27 1.27)) hide)))
+                    (size 1.27 1.27)) hide))
+        (property "Manufacturer" "N/A"
+            (id 4)
+            (at 220.345 90.1699 0)
+            (effects
+                (font
+                    (size 1.27 1.27))
+                (justify left) hide))
+        (property "MfgPartNo" "N/A"
+            (id 5)
+            (at 220.345 92.7099 0)
+            (effects
+                (font
+                    (size 1.27 1.27))
+                (justify left) hide))
+        (property "Vendor" "N/A"
+            (id 6)
+            (at 220.345 95.2499 0)
+            (effects
+                (font
+                    (size 1.27 1.27))
+                (justify left) hide))
+        (property "VendorPartNo" "N/A"
+            (id 7)
+            (at 220.345 97.7899 0)
+            (effects
+                (font
+                    (size 1.27 1.27))
+                (justify left) hide)))
     (symbol
         (lib_id "power:GND")
