File: ddr3l.kicad_sch (KiCad schematic)
At the start: 35 parts, among them U4 MCIMX6Y2DVM09AB, U6 IS43TR16256BL-107MBL

Commit message: Update fields
Parts:
- C43, C44, C45, C46, C47, C52, C53, C56, C57, C58, C59, C60, C61, C62, C63, C64, C65, C66: Manufacturer (none) -> Samsung Electro-Mechanics; MfgPartNo (none) -> CL05A224KQ5NNNC; Vendor (none) -> Digi-Key; VendorPartNo (none) -> 1276-1124-1-ND
- C48: Manufacturer (none) -> Samsung Electro-Mechanics; MfgPartNo (none) -> CL21A106KPFNNNG; Vendor (none) -> Digi-Key; VendorPartNo (none) -> 1276-6456-1-ND
- C49, C50: Manufacturer (none) -> Samsung Electro-Mechanics; MfgPartNo (none) -> CL05C2R2CB51PNC; Vendor (none) -> Digi-Key; VendorPartNo (none) -> 1276-CL05C2R2CB51PNCCT-ND
- C51: Manufacturer (none) -> Samsung Electro-Mechanics; MfgPartNo (none) -> CL10A475KQ8NNNC; Vendor (none) -> Digi-Key; VendorPartNo (none) -> 1276-1045-1-ND
- C54, C55: Manufacturer (none) -> Murata Electronics; MfgPartNo (none) -> GRM155R71H104KE14D; Vendor (none) -> Digi-Key; VendorPartNo (none) -> 490-10700-1-ND
- R13, R15, R17: Manufacturer (none) -> YAGEO; MfgPartNo (none) -> RC0402JR-0710KL; Vendor (none) -> Digi-Key; VendorPartNo (none) -> 311-10KJRCT-ND
- R14, R21: Manufacturer (none) -> YAGEO; MfgPartNo (none) -> RC0402FR-07240RL; Vendor (none) -> Digi-Key; VendorPartNo (none) -> 311-240LRCT-ND
- R16: Manufacturer (none) -> YAGEO; MfgPartNo (none) -> RT0402FRE07470RL; Vendor (none) -> Digi-Key; VendorPartNo (none) -> 13-RT0402FRE07470RLCT-ND
- R18, R19: Manufacturer (none) -> YAGEO; MfgPartNo (none) -> RC0402FR-131K5L; Vendor (none) -> Digi-Key; VendorPartNo (none) -> 13-RC0402FR-131K5LCT-ND
- R20: Manufacturer (none) -> N/A; MfgPartNo (none) -> N/A; Vendor (none) -> N/A; VendorPartNo (none) -> N/A
- U6: Manufacturer (none) -> ISSI; MfgPartNo (none) -> IS43TR16256BL-107MBL; Vendor (none) -> Digi-Key; VendorPartNo (none) -> 706-1729-ND
