File: nand.kicad_sch (KiCad schematic)
At the start: 14 parts, among them U4 MCIMX6Y2DVM09AB, U7 MT29F4G08ABAEAH4

Commit message: Update fields
Parts:
- C67: Manufacturer (none) -> Samsung Electro-Mechanics; MfgPartNo (none) -> CL05A224KQ5NNNC; Vendor (none) -> Digi-Key; VendorPartNo (none) -> 1276-1124-1-ND
- C68: Manufacturer (none) -> YAGEO; MfgPartNo (none) -> CC0402JRNPO9BN180; Vendor (none) -> Digi-Key; VendorPartNo (none) -> 311-1415-1-ND
- C69: Manufacturer (none) -> Samsung Electro-Mechanics; MfgPartNo (none) -> CL10A475KQ8NNNC; Vendor (none) -> Digi-Key; VendorPartNo (none) -> 1276-1045-1-ND
- C70, C71, C72, C73: Manufacturer (none) -> Murata Electronics; MfgPartNo (none) -> GRM155R71H104KE14D; Vendor (none) -> Digi-Key; VendorPartNo (none) -> 490-10700-1-ND
- R22: Manufacturer (none) -> General; MfgPartNo (none) -> General; Vendor (none) -> General; VendorPartNo (none) -> General
- R23, R24: Manufacturer (none) -> TE Connectivity; MfgPartNo (none) -> CRGP0402F10R; Vendor (none) -> Digi-Key; VendorPartNo (none) -> A130331CT-ND
- R25, R26: Manufacturer (none) -> YAGEO; MfgPartNo (none) -> RC0402JR-0710KL; Vendor (none) -> Digi-Key; VendorPartNo (none) -> 311-10KJRCT-ND
- U7: Manufacturer (none) -> Micron Technology, Inc; MfgPartNo (none) -> MT29F4G08ABAEAH4:E TR; Vendor (none) -> Digi-Key; VendorPartNo (none) -> 557-1871-1-ND
