File: regulators.kicad_sch (KiCad schematic)
At the start: 33 parts, among them U1 MP2143DJ, U2 AP22615AWU-7, U3 LMR10510XMF

Commit message: Update fields
Parts:
- C1, C12, C2, C3, C5, C7: Manufacturer (none) -> Samsung Electro-Mechanics; MfgPartNo (none) -> CL21A106KPFNNNG; Vendor (none) -> Digi-Key; VendorPartNo (none) -> 1276-6456-1-ND
- C10, C14, C6: Manufacturer (none) -> Murata Electronics; MfgPartNo (none) -> GRM155R71H104KE14D; Vendor (none) -> Digi-Key; VendorPartNo (none) -> 490-10700-1-ND
- C11, C13: Manufacturer (none) -> Murata Electronics; MfgPartNo (none) -> GRM21BR61A226ME51L; Vendor (none) -> Digi-Key; VendorPartNo (none) -> 490-10511-1-ND
- C4: Manufacturer (none) -> TDK Corporation; MfgPartNo (none) -> CGB2A1X5R1E105K033BC; Vendor (none) -> Digi-Key; VendorPartNo (none) -> 445-13185-1-ND
- C8: Manufacturer (none) -> Samsung Electro-Mechanics; MfgPartNo (none) -> CL05A224KQ5NNNC; Vendor (none) -> Digi-Key; VendorPartNo (none) -> 1276-1124-1-ND
- C9, TP1, TP2, TP3, TP4, TP5: Manufacturer (none) -> N/A; MfgPartNo (none) -> N/A; Vendor (none) -> N/A; VendorPartNo (none) -> N/A
- D1: Manufacturer (none) -> SMC Diode Solutions; MfgPartNo (none) -> 1N5819W; Vendor (none) -> Digi-Key; VendorPartNo (none) -> 1655-1N5819WCT-ND
- L1: Manufacturer (none) -> Wurth; MfgPartNo (none) -> 74438336010; Vendor (none) -> Digi-Key; VendorPartNo (none) -> 732-5693-1-ND
- L2: Manufacturer (none) -> Murata Electronics; MfgPartNo (none) -> 1255AY-3R9N=P3; Vendor (none) -> Digi-Key; VendorPartNo (none) -> 490-14062-1-ND
- R1, R2: Manufacturer (none) -> YAGEO; MfgPartNo (none) -> RC0402FR-07100KL; Vendor (none) -> Digi-Key; VendorPartNo (none) -> 311-100KLRCT-ND
- R3: Manufacturer (none) -> YAGEO; MfgPartNo (none) -> RC0402JR-0710KL; Vendor (none) -> Digi-Key; VendorPartNo (none) -> 311-10KJRCT-ND
- R4: Manufacturer (none) -> Panasonic Electronic; MfgPartNo (none) -> ERJ-2RKF3401X; Vendor (none) -> Digi-Key; VendorPartNo (none) -> P3.40KLCT-ND
- R5: value 200k 0603 1% -> 200k 0402 1%; footprint Resistor_SMD:R_0603_1608Metric -> Resistor_SMD:R_0402_1005Metric; Manufacturer (none) -> YAGEO; MfgPartNo (none) -> RC0402FR-07200KL; Vendor (none) -> Digi-Key; VendorPartNo (none) -> 311-200KLRCT-ND
- R6: Manufacturer (none) -> Vishay Dale; MfgPartNo (none) -> CRCW040244K2FKEDC; Vendor (none) -> Digi-Key; VendorPartNo (none) -> 541-4106-1-ND
- R7: Manufacturer (none) -> YAGEO; MfgPartNo (none) -> RC0402FR-0712K4L; Vendor (none) -> Digi-Key; VendorPartNo (none) -> 311-12.4KLRCT-ND
- R8: Manufacturer (none) -> YAGEO; MfgPartNo (none) -> RC0402FR-0710KP; Vendor (none) -> Digi-Key; VendorPartNo (none) -> YAG1249CT-ND
- U1: Manufacturer (none) -> Monolithic Power Systems; MfgPartNo (none) -> MP2143DJ-LF-Z; Vendor (none) -> Digi-Key; VendorPartNo (none) -> 1589-1874-1-ND
- U2: Manufacturer (none) -> Diodes Incorporated; MfgPartNo (none) -> AP22615AWU-7; Vendor (none) -> Digi-Key; VendorPartNo (none) -> AP22615AWU-7DICT-ND
- U3: Manufacturer (none) -> Texas Instruments; MfgPartNo (none) -> LMR10510XMF/NOPB; Vendor (none) -> Digi-Key; VendorPartNo (none) -> 296-38159-1-ND

Commit message: KiCad 7
Parts:
- R5: value 200k 0402 1% -> 200k 0603 1%; footprint Resistor_SMD:R_0402_1005Metric -> Resistor_SMD:R_0603_1608Metric
