File: ethernet.kicad_sch (KiCad schematic)
At the start: 35 parts, among them J3 TE_1888250-1, T1 H1102, U4 MCIMX6Y2DVM09AB, U8 LAN8700C-AEZG

Commit message: Fix grid
Changed lines of the file:
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@@
   (junction (at 195.58 104.14) (diameter 0) (color 0 0 0 0)
   )
-  (junction (at 178.435 69.85) (diameter 0) (color 0 0 0 0)
-  )
   (junction (at 172.72 107.95) (diameter 0) (color 0 0 0 0)
   )
@@
   )
   (junction (at 160.02 182.88) (diameter 0) (color 0 0 0 0)
+  )
+  (junction (at 179.07 69.85) (diameter 0) (color 0 0 0 0)
   )
   (junction (at 411.48 161.29) (diameter 0) (color 0 0 0 0)
@@
     (stroke (width 0) (type default))
   )
-  (wire (pts (xy 178.435 69.85) (xy 186.69 69.85))
+  (wire (pts (xy 157.48 69.85) (xy 179.07 69.85))
     (stroke (width 0) (type default))
   )
@@
     (stroke (width 0) (type default))
   )
+  (wire (pts (xy 179.07 69.85) (xy 186.69 69.85))
+    (stroke (width 0) (type default))
+  )
   (wire (pts (xy 105.41 111.76) (xy 105.41 144.78))
     (stroke (width 0) (type default))
@@
   )
   (wire (pts (xy 66.04 114.3) (xy 87.63 114.3))
-    (stroke (width 0) (type default))
-  )
-  (wire (pts (xy 157.48 69.85) (xy 178.435 69.85))
     (stroke (width 0) (type default))
   )
@@
     )
   )
-  (symbol (lib_id "power:PWR_FLAG") (at 178.435 69.85 0) (unit 1)
-    (in_bom yes) (on_board yes) (dnp no) (fields_autoplaced)
-    (property "Reference" "#FLG0102" (at 178.435 67.945 0)
-      (effects (font (size 1.27 1.27)) hide)
-    )
-    (property "Value" "PWR_FLAG" (at 178.435 64.77 0)
-      (effects (font (size 1.27 1.27)))
-    )
-    (property "Footprint" "" (at 178.435 69.85 0)
-      (effects (font (size 1.27 1.27)) hide)
-    )
-    (property "Datasheet" "~" (at 178.435 69.85 0)
-      (effects (font (size 1.27 1.27)) hide)
-    )
+  (symbol (lib_id "power:PWR_FLAG") (at 179.07 69.85 0) (unit 1)
+    (in_bom yes) (on_board yes) (dnp no) (fields_autoplaced)
+    (property "Reference" "#FLG0102" (at 179.07 67.945 0)
+      (effects (font (size 1.27 1.27)) hide)
+    )
+    (property "Value" "PWR_FLAG" (at 179.07 64.77 0)
+      (effects (font (size 1.27 1.27)))
+    )
+    (property "Footprint" "" (at 179.07 69.85 0)
+      (effects (font (size 1.27 1.27)) hide)
+    )
+    (property "Datasheet" "~" (at 179.07 69.85 0)
+      (effects (font (size 1.27 1.27)) hide)
+    )
